File: Holding-Cabinet-Hardware.kicad_sch (KiCad schematic)
At the start: 0 parts

Commit message: Update
Other:
- sheet Heater ports: added +5V, GND, IN1, IN2, IN3, IN4; removed none
- sheet LCD 16x2 Display ports: added +5V, GND, I2C2_SCL, I2C2_SDA; removed none
- sheet MCU ports: added I2C2_SDA; removed none
Changed lines of the file:
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@@
 	)
 	(sheet
-		(at 111.76 58.42)
-		(size 17.78 6.35)
+		(at 86.36 91.44)
+		(size 24.13 35.56)
 		(exclude_from_sim no)
 		(in_bom yes)
@@
 		)
 		(property "Sheetname" "Heater"
-			(at 111.76 57.7084 0)
+			(at 86.36 90.7284 0)
 			(show_name no)
 			(do_not_autoplace no)
@@
 		)
 		(property "Sheetfile" "heater.kicad_sch"
-			(at 111.76 65.3546 0)
+			(at 86.36 127.5846 0)
 			(show_name no)
 			(do_not_autoplace no)
@@
 				)
 				(justify left top)
+			)
+		)
+		(pin "+5V" input
+			(at 86.36 99.06 180)
+			(effects
+				(font
+					(size 1.27 1.27)
+				)
+				(justify left)
+			)
+		)
+		(pin "GND" input
+			(at 86.36 109.22 180)
+			(effects
+				(font
+					(size 1.27 1.27)
+				)
+				(justify left)
+			)
+		)
+		(pin "IN1" input
+			(at 86.36 113.03 180)
+			(effects
+				(font
+					(size 1.27 1.27)
+				)
+				(justify left)
+			)
+		)
+		(pin "IN2" input
+			(at 86.36 116.84 180)
+			(effects
+				(font
+					(size 1.27 1.27)
+				)
+				(justify left)
+			)
+		)
+		(pin "IN3" input
+			(at 92.71 127 270)
+			(effects
+				(font
+					(size 1.27 1.27)
+				)
+				(justify left)
+			)
+		)
+		(pin "IN4" input
+			(at 96.52 127 270)
+			(effects
+				(font
+					(size 1.27 1.27)
+				)
+				(justify left)
 			)
 		)
@@
 			)
 		)
-		(pin "IN1" output
+		(pin "IN1" input
 			(at 33.02 101.6 180)
 			(effects
@@
 			)
 		)
-		(pin "IN2" output
+		(pin "IN2" input
 			(at 33.02 104.14 180)
 			(effects
@@
 			)
 		)
-		(pin "IN3" output
+		(pin "IN3" input
 			(at 33.02 106.68 180)
 			(effects
@@
 			)
 		)
-		(pin "IN4" output
+		(pin "IN4" input
 			(at 33.02 109.22 180)
 			(effects
@@
 			)
 		)
-		(pin "LED3" output
+		(pin "LED3" input
 			(at 78.74 102.87 0)
 			(effects
@@
 			)
 		)
-		(pin "LED2" output
+		(pin "LED2" input
 			(at 78.74 105.41 0)
 			(effects
@@
 			)
 		)
-		(pin "LED1" output
+		(pin "LED1" input
 			(at 78.74 107.95 0)
 			(effects
@@
 				)
 				(justify right)
+			)
+		)
+		(pin "I2C2_SDA" input
+			(at 33.02 113.03 180)
+			(effects
+				(font
+					(size 1.27 1.27)
+				)
+				(justify left)
 			)
 		)
@@
 	)
 	(sheet
-		(at 158.75 91.44)
-		(size 57.15 34.29)
+		(at 121.92 92.71)
+		(size 22.86 34.29)
 		(exclude_from_sim no)
 		(in_bom yes)
@@
 		)
 		(property "Sheetname" "LCD 16x2 Display"
-			(at 158.75 90.7284 0)
+			(at 121.92 91.9984 0)
 			(show_name no)
 			(do_not_autoplace no)
@@
 		)
 		(property "Sheetfile" "lcd_16_2_display.kicad_sch"
-			(at 158.75 126.3146 0)
+			(at 121.92 127.5846 0)
 			(show_name no)
 			(do_not_autoplace no)
@@
 			)
 		)
+		(pin "+5V" input
+			(at 121.92 96.52 180)
+			(effects
+				(font
+					(size 1.27 1.27)
+				)
+				(justify left)
+			)
+		)
+		(pin "GND" input
+			(at 121.92 100.33 180)
+			(effects
+				(font
+					(size 1.27 1.27)
+				)
+				(justify left)
+			)
+		)
+		(pin "I2C2_SCL" input
+			(at 121.92 105.41 180)
+			(effects
+				(font
+					(size 1.27 1.27)
+				)
+				(justify left)
+			)
+		)
+		(pin "I2C2_SDA" input
+			(at 121.92 109.22 180)
+			(effects
+				(font
+					(size 1.27 1.27)
+				)
+				(justify left)
+			)
+		)
