File: heater.kicad_sch (KiCad schematic)
At the start: 0 parts

Commit message: Added Silicone heating pad and related circuitry
Parts:
- added D1: 1N4001, Diode_THT:D_DO-41_SOD81_P10.16mm_Horizontal, symbol Diode:1N4001
- added F1: Fuse, symbol Device:Fuse
- added K1: SRD-05VDC-SL-C, Relay_THT:Relay_SPDT_SANYOU_SRD_Series_Form_C, symbol Relay:SANYOU_SRD_Form_C
- added Q1: 2N3904, Package_TO_SOT_THT:TO-92_Inline, symbol Transistor_BJT:2N3904
- added R1: Silicone Heating Pad 120VAC, 300W, symbol Device:Heater
- added R2, R3: R_US, symbol Device:R_US
- added SW1: SW_SPST, symbol Switch:SW_SPST
Connections:
- new net: F1.2, K1.1
- new net: D1.2 (A), K1.2, Q1.3 (C)
- new net: K1.3, R1.1
- new net: D1.1 (K), K1.5, R2.2
- new net: F1.1, SW1.2 (B)
- new net: Q1.2 (B), R3.2
- new net GND: Q1.1 (E)
- new net VCC: R2.1

Commit message: Update
Parts:
- added J2: Conn_01x06_Pin, symbol Connector:Conn_01x06_Pin
Connections:
- net GND: now also J2.1 (Pin_1)
- net AC Nuetral: now reaches R1.2
- net AC Hot: now reaches SW1.1 (A)
- new net +5V: J2.6 (Pin_6)
- new net IN1: J2.2 (Pin_2)
- new net IN2: J2.3 (Pin_3)
- new net IN3: J2.4 (Pin_4)
- new net IN4: J2.5 (Pin_5)
Other:
- note added: "High Voltage Area"
- moved on the sheet: D1, F1, K1, Q1, R1, R2, R3, SW1

Commit message: Update
Parts:
- removed D1: 1N4001, Diode_THT:D_DO-41_SOD81_P10.16mm_Horizontal, symbol Diode:1N4001
- removed F1: Fuse, symbol Device:Fuse
- removed K1: SRD-05VDC-SL-C, Relay_THT:Relay_SPDT_SANYOU_SRD_Series_Form_C, symbol Relay:SANYOU_SRD_Form_C
- removed Q1: 2N3904, Package_TO_SOT_THT:TO-92_Inline, symbol Transistor_BJT:2N3904
- removed R1: Silicone Heating Pad 120VAC, 300W, symbol Device:Heater
- removed R2, R3: R_US, symbol Device:R_US
- removed SW1: SW_SPST, symbol Switch:SW_SPST
Other:
- note removed: "High Voltage Area"
