File: lcd_16_2_display.kicad_sch (KiCad schematic)
At the start: 0 parts

Commit message: Added connector for pinout
Parts:
- added J1: Conn_01x04_Pin, symbol Connector:Conn_01x04_Pin
Connections:
- new net +5V: J1.1 (Pin_1)
- new net GND: J1.4 (Pin_4)

Commit message: Updates
Connections:
- net +5V: now also J1.2 (Pin_2); no longer J1.1 (Pin_1)
- net GND: now also J1.1 (Pin_1); no longer J1.4 (Pin_4)
- net I2C_SDA: now reaches J1.3 (Pin_3)
- new net I2C_SCL: J1.4 (Pin_4)

Commit message: Update
Connections:
- net I2C_SCL renamed I2C2_SCL
- net I2C_SDA renamed I2C2_SDA
Changed lines of the file:
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@@
 		)
 	)
-	(hierarchical_label "I2C_SDA"
+	(hierarchical_label "I2C2_SDA"
 		(shape input)
 		(at 93.98 87.63 180)
@@
 		)
 	)
-	(hierarchical_label "I2C_SCL"
+	(hierarchical_label "I2C2_SCL"
 		(shape input)
 		(at 93.98 85.09 180)
