File: mcu.kicad_sch (KiCad schematic)
At the start: 0 parts

Commit message: Updated sheet connections for MCU to Display
Parts:
- added U1: STM32L476RGTx, Package_QFP:LQFP-64_10x10mm_P0.5mm, symbol MCU_ST_STM32L4:STM32L476RGTx
Connections:
- new net: U1.18 (VSS), U1.31 (VSS), U1.47 (VSS), U1.63 (VSS)
- new net TCK: U1.49 (PA14)
- new net TMS: U1.46 (PA13)
- new net USART_RX: U1.17 (PA3)
- new net USART_TX: U1.16 (PA2)
- new net User Button: U1.2 (PC13)
- new net User LED: U1.21 (PA5)
- new net digit_cc1: U1.26 (PB0)
- new net digit_cc2: U1.27 (PB1)
- new net digit_cc3: U1.28 (PB2)
- new net digit_cc4: U1.55 (PB3)
- new net segment_a: U1.8 (PC0)
- new net segment_b: U1.9 (PC1)
- new net segment_c: U1.10 (PC2)
- new net segment_d: U1.11 (PC3)
- new net segment_dpx: U1.38 (PC7)
- new net segment_e: U1.24 (PC4)
- new net segment_f: U1.25 (PC5)
- new net segment_g: U1.37 (PC6)

Commit message: Update
Connections:
- net I2C2_SCL: now reaches U1.29 (PB10)
- net I2C2_SDA: now reaches U1.30 (PB11)
- net IN3: now reaches U1.39 (PC8)
- net IN4: now reaches U1.40 (PC9)
- net LED1: now reaches U1.41 (PA8)
- net LED2: now reaches U1.42 (PA9)
- net LED3: now reaches U1.43 (PA10)
- net SW1: now reaches U1.56 (PB4)
- net SW2: now reaches U1.57 (PB5)
- net SW3: now reaches U1.58 (PB6)
- net SW4: now reaches U1.59 (PB7)
- net digit_cc1: no longer names the net of U1.26 (PB0)
- net digit_cc2: no longer names the net of U1.27 (PB1)
- net digit_cc3: no longer names the net of U1.28 (PB2)
- net digit_cc4: no longer names the net of U1.55 (PB3)
- net segment_a: no longer names the net of U1.8 (PC0)
- net segment_b: no longer names the net of U1.9 (PC1)
- net segment_c: no longer names the net of U1.10 (PC2)
- net segment_d: no longer names the net of U1.11 (PC3)
- net segment_dpx renamed IN2
- net segment_e: no longer names the net of U1.24 (PC4)
- net segment_f: no longer names the net of U1.25 (PC5)
- net segment_g renamed IN1
Changed lines of the file:
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@@
-	(wire
-		(pts
-			(xy 111.76 87.63) (xy 113.03 87.63)
-		)
-		(stroke
-			(width 0)
-			(type default)
-		)
-	)
 	(wire
 		(pts
@@
 	(wire
 		(pts
-			(xy 111.76 80.01) (xy 113.03 80.01)
-		)
-		(stroke
-			(width 0)
-			(type default)
-		)
-	)
-	(wire
-		(pts
-			(xy 111.76 82.55) (xy 113.03 82.55)
+			(xy 149.86 74.93) (xy 148.59 74.93)
 		)
 		(stroke
@@
 	(wire
 		(pts
+			(xy 151.13 123.19) (xy 148.59 123.19)
+		)
+		(stroke
+			(width 0)
+			(type default)
+		)
+	)
+	(wire
+		(pts
 			(xy 148.59 90.17) (xy 171.45 90.17)
 		)
@@
 	(wire
 		(pts
+			(xy 111.76 95.25) (xy 113.03 95.25)
+		)
+		(stroke
+			(width 0)
+			(type default)
+		)
+	)
+	(wire
+		(pts
 			(xy 149.86 105.41) (xy 148.59 105.41)
 		)
@@
 	(wire
 		(pts
+			(xy 149.86 113.03) (xy 148.59 113.03)
+		)
+		(stroke
+			(width 0)
+			(type default)
+		)
+	)
+	(wire
+		(pts
 			(xy 97.79 110.49) (xy 113.03 110.49)
 		)
@@
 	(wire
 		(pts
-			(xy 111.76 95.25) (xy 113.03 95.25)
-		)
-		(stroke
-			(width 0)
-			(type default)
-		)
-	)
-	(wire
-		(pts
-			(xy 111.76 85.09) (xy 113.03 85.09)
+			(xy 149.86 80.01) (xy 148.59 80.01)
+		)
+		(stroke
+			(width 0)
+			(type default)
+		)
+	)
+	(wire
+		(pts
+			(xy 151.13 125.73) (xy 148.59 125.73)
+		)
+		(stroke
+			(width 0)
+			(type default)
+		)
+	)
+	(wire
+		(pts
+			(xy 111.76 97.79) (xy 113.03 97.79)
+		)
+		(stroke
+			(width 0)
+			(type default)
+		)
+	)
+	(wire
+		(pts
+			(xy 149.86 77.47) (xy 148.59 77.47)
+		)
+		(stroke
+			(width 0)
+			(type default)
+		)
+	)
+	(wire
+		(pts
+			(xy 149.86 115.57) (xy 148.59 115.57)
 		)
 		(stroke
@@
 	(wire
 		(pts
+			(xy 149.86 110.49) (xy 148.59 110.49)
+		)
+		(stroke
+			(width 0)
+			(type default)
+		)
+	)
+	(wire
+		(pts
+			(xy 111.76 92.71) (xy 113.03 92.71)
+		)
+		(stroke
+			(width 0)
+			(type default)
+		)
+	)
+	(wire
+		(pts
 			(xy 149.86 97.79) (xy 148.59 97.79)
 		)
@@
 	(wire
 		(pts
-			(xy 111.76 92.71) (xy 113.03 92.71)
-		)
-		(stroke
-			(width 0)
-			(type default)
-		)
-	)
-	(wire
-		(pts
-			(xy 111.76 77.47) (xy 113.03 77.47)
-		)
-		(stroke
-			(width 0)
-			(type default)
-		)
-	)
-	(wire
-		(pts
-			(xy 111.76 90.17) (xy 113.03 90.17)
+			(xy 111.76 100.33) (xy 113.03 100.33)
+		)
+		(stroke
+			(width 0)
+			(type default)
+		)
+	)
+	(wire
+		(pts
+			(xy 149.86 107.95) (xy 148.59 107.95)
 		)
 		(stroke
@@
 		)
 	)
-	(hierarchical_label "digit_cc2"
-		(shape input)
-		(at 149.86 100.33 0)
-		(effects
-			(font
-				(size 1.27 1.27)
-			)
-			(justify left)
-		)
-	)
-	(hierarchical_label "digit_cc4"
-		(shape input)
-		(at 149.86 105.41 0)
-		(effects
-			(font
-				(size 1.27 1.27)
-			)
-			(justify left)
-		)
-	)
-	(hierarchical_label "segment_dpx"
+	(hierarchical_label "LED2"
+		(shape input)
+		(at 149.86 77.47 0)
+		(effects
+			(font
+				(size 1.27 1.27)
+			)
+			(justify left)
+		)
+	)
+	(hierarchical_label "I2C2_SDA"
+		(shape input)
+		(at 151.13 125.73 0)
+		(effects
+			(font
+				(size 1.27 1.27)
+			)
+			(justify left)
+		)
+	)
+	(hierarchical_label "IN3"
+		(shape input)
+		(at 111.76 97.79 180)
+		(effects
+			(font
+				(size 1.27 1.27)
+			)
+			(justify right)
+		)
+	)
+	(hierarchical_label "LED1"
+		(shape input)
+		(at 149.86 74.93 0)
+		(effects
+			(font
+				(size 1.27 1.27)
+			)
+			(justify left)
+		)
+	)
+	(hierarchical_label "IN4"
+		(shape input)
+		(at 111.76 100.33 180)
+		(effects
+			(font
+				(size 1.27 1.27)
+			)
+			(justify right)
+		)
+	)
+	(hierarchical_label "LED3"
+		(shape input)
+		(at 149.86 80.01 0)
+		(effects
+			(font
+				(size 1.27 1.27)
+			)
+			(justify left)
+		)
+	)
+	(hierarchical_label "IN2"
 		(shape input)
 		(at 111.76 95.25 180)
@@
 		)
 	)
-	(hierarchical_label "digit_cc3"
-		(shape input)
-		(at 149.86 102.87 0)
-		(effects
-			(font
-				(size 1.27 1.27)
-			)
-			(justify left)
-		)
-	)
-	(hierarchical_label "segment_c"
-		(shape input)
-		(at 111.76 82.55 180)
+	(hierarchical_label "IN1"
+		(shape input)
+		(at 111.76 92.71 180)
 		(effects
 			(font
@@
 		)
 	)
-	(hierarchical_label "segment_b"
-		(shape input)
-		(at 111.76 80.01 180)
-		(effects
-			(font
-				(size 1.27 1.27)
-			)
-			(justify right)
-		)
-	)
-	(hierarchical_label "segment_g"
-		(shape input)
-		(at 111.76 92.71 180)
-		(effects
-			(font
-				(size 1.27 1.27)
-			)
-			(justify right)
-		)
-	)
-	(hierarchical_label "segment_f"
-		(shape input)
-		(at 111.76 90.17 180)
-		(effects
-			(font
-				(size 1.27 1.27)
-			)
-			(justify right)
-		)
-	)
-	(hierarchical_label "digit_cc1"
-		(shape input)
-		(at 149.86 97.79 0)
-		(effects
-			(font
-				(size 1.27 1.27)
-			)
-			(justify left)
-		)
-	)
-	(hierarchical_label "segment_a"
-		(shape input)
-		(at 111.76 77.47 180)
-		(effects
-			(font
-				(size 1.27 1.27)
-			)
-			(justify right)
-		)
-	)
-	(hierarchical_label "segment_d"
-		(shape input)
-		(at 111.76 85.09 180)
-		(effects
-			(font
-				(size 1.27 1.27)
-			)
-			(justify right)
-		)
-	)
-	(hierarchical_label "segment_e"
-		(shape input)
-		(at 111.76 87.63 180)
-		(effects
-			(font
-				(size 1.27 1.27)
-			)
-			(justify right)
-		)
-	)
+	(hierarchical_label "I2C2_SCL"
+		(shape input)
+		(at 151.13 123.19 0)
+		(effects
+			(font
+				(size 1.27 1.27)
+			)
+			(justify left)
+		)
+	)
+	(hierarchical_label "SW1"
+		(shape input)
+		(at 149.86 107.95 0)
+		(effects
+			(font
+				(size 1.27 1.27)
+			)
+			(justify left)
+		)
+	)
+	(hierarchical_label "SW3"
+		(shape input)
+		(at 149.86 113.03 0)
+		(effects
+			(font
+				(size 1.27 1.27)
+			)
+			(justify left)
+		)
+	)
+	(hierarchical_label "SW4"
+		(shape input)
+		(at 149.86 115.57 0)
+		(effects
+			(font
+				(size 1.27 1.27)
+			)
+			(justify left)
+		)
+	)
+	(hierarchical_label "SW2"
+		(shape input)
+		(at 149.86 110.49 0)
+		(effects
+			(font
+				(size 1.27 1.27)
+			)
+			(justify left)
+		)
+	)
