File: sensing.kicad_sch (KiCad schematic)
At the start: 0 parts

Commit message: Added NTC specs
Parts:
- added R1: 10K, 1%, MF, symbol Device:R_US
- added TH1: Thermistor_NTC, symbol Device:Thermistor_NTC
Connections:
- new net +3.3V: R1.1
- new net GND: TH1.2
- new net NTC_A_D: R1.2, TH1.1
